File: pcb/Display_RP2350.kicad_pcb (KiCad board)
At the start: 4 copper layers, 32.1 x 39.1 mm, 57 parts, among them J1 USB_C_Receptacle_USB2.0_16P, J2 Screw_Terminal_01x03, J3 PicoBlade F 1x7, J4 SM03B-SRSS-TB, SW1 SW_Push, SW2 SW_Push, U1 RP2350_60QFN, U2 TLVM365R15RDNR, U3 W25Q32RVXHJQ, U4 TCAN332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

Commit message: PCB updates
Parts:
- added H1: MountingHole, MountingHole:MountingHole_2.2mm_M2_ISO14580, F.Cu at (94.1, 87.5)
- moved C4 2.04 mm to (94.1, 84.2), turned to 180 degrees
- moved C11 1.02 mm to (111.1, 95.6)
- moved R1 1.02 mm to (111.1, 94.5)
- moved D2 1.02 mm to (110.1, 92.8)
- moved F1 0.76 mm to (114.7, 92.7)
- moved D1 0.69 mm to (114.6, 95.6)
- moved U4 0.64 mm to (111.1, 98.7)
- moved C24 0.64 mm to (108.0, 98.7)
- moved C12 0.51 mm to (118.2, 100.5)
Routing:
- net GND: track 110.1 -> 112.0 mm
- net +12V: track 14.2 -> 15.0 mm
- net VBUS: track 25.9 -> 26.6 mm
- net CANH: track 12.8 -> 13.4 mm
- net GMLAN_CAN_TX: track 7.51 -> 6.95 mm
Other:
- board text added: "ACC (+)"
- board text added: "GMLAN"
- board text added: "GND"
- board text added: "LOW SPEED GMLAN MESSAGE DISPLAY J-S.DEV"
