File: pcb/Display_RP2350.kicad_sch (KiCad schematic)
At the start: 57 parts, among them J1 USB_C_Receptacle_USB2.0_16P, J2 Screw_Terminal_01x03, J3 PicoBlade F 1x7, J4 SM03B-SRSS-TB, SW1 SW_Push, SW2 SW_Push, U1 RP2350_60QFN, U2 TLVM365R15RDNR, U3 W25Q32RVXHJQ, U4 TCAN332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

Commit message: PCB updates
Parts:
- added H1: MountingHole, MountingHole:MountingHole_2.2mm_M2_ISO14580, symbol Mechanical:MountingHole
Changed lines of the file:
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@@
+	)
+	(symbol
+		(lib_id "Mechanical:MountingHole")
+		(at 266.7 203.2 0)
+		(unit 1)
+		(exclude_from_sim yes)
+		(in_bom no)
+		(on_board yes)
+		(dnp no)
+		(fields_autoplaced yes)
+		(property "Reference" "H1"
+			(at 269.24 201.9299 0)
+			(effects
+				(font
+					(size 1.27 1.27)
+				)
+				(justify left)
+			)
+		)
+		(property "Value" "MountingHole"
+			(at 269.24 204.4699 0)
+			(effects
+				(font
+					(size 1.27 1.27)
+				)
+				(justify left)
+			)
+		)
+		(property "Footprint" "MountingHole:MountingHole_2.2mm_M2_ISO14580"
+			(at 266.7 203.2 0)
+			(effects
+				(font
+					(size 1.27 1.27)
+				)
+				(hide yes)
+			)
+		)
+		(property "Datasheet" "~"
+			(at 266.7 203.2 0)
+			(effects
+				(font
+					(size 1.27 1.27)
+				)
+				(hide yes)
+			)
+		)
+		(property "Description" "Mounting Hole without connection"
+			(at 266.7 203.2 0)
+			(effects
+				(font
+					(size 1.27 1.27)
+				)
+				(hide yes)
+			)
+		)
+		(instances
+			(project ""
+				(path "/94683f5c-9cd9-448e-be96-9792537b5cb8"
+					(reference "H1")
+					(unit 1)
+				)
+			)
+		)
 	)
 	(symbol
